File: Avrille/64_Outs/64_Outs.kicad_sch (KiCad schematic)
At the start: 70 parts, among them J1 POWER, J2 Midi-In, J3 Midi-Thru, J4 ICSP, J5 FT232, J6 Expr 2, J7 Expr 1, Q1 BC337, SW1 RESET, SW2 Prog, SW3 Channel, U1 74HC14, U2 6N138, U3 TMR 6-2411, U4 PIC18F26K80, U5 LM358

Commit message: Update to SMD Version
Parts:
- removed C5: 100n, Capacitor_THT:C_Disc_D4.3mm_W1.9mm_P5.00mm, symbol Device:C_Small
- removed H10, H11, H12, H8, H9: MountingHole, MountingHole:MountingHole_3.2mm_M3, symbol Mechanical:MountingHole
- removed J6: Expr 2, Connector_PinHeader_2.54mm:PinHeader_1x02_P2.54mm_Vertical, symbol Connector:Screw_Terminal_01x02
- removed J7: Expr 1, Connector_PinHeader_2.54mm:PinHeader_1x02_P2.54mm_Vertical, symbol Connector:Screw_Terminal_01x02
- removed R16, R17: 10, Resistor_THT:R_Axial_DIN0207_L6.3mm_D2.5mm_P10.16mm_Horizontal, symbol Device:R
- removed U5: LM358, Package_DIP:CERDIP-8_W7.62mm_SideBrazed_Socket, symbol Amplifier_Operational:LM358
- added TP6: GND, TestPoint:TestPoint_Loop_D2.50mm_Drill1.0mm, symbol Connector:TestPoint
- C1: footprint Capacitor_THT:C_Disc_D4.3mm_W1.9mm_P5.00mm -> Capacitor_THT:C_Disc_D5.0mm_W2.5mm_P2.50mm
- C2: footprint (none) -> Capacitor_THT:CP_Radial_D6.3mm_P2.50mm
- C3: renamed from C14; footprint Capacitor_THT:C_Disc_D4.3mm_W1.9mm_P5.00mm -> Capacitor_THT:C_Disc_D5.0mm_W2.5mm_P2.50mm
- C4: renamed from C3; footprint (none) -> Capacitor_THT:CP_Radial_D5.0mm_P2.00mm
- C5: renamed from C4; footprint Capacitor_THT:C_Disc_D4.3mm_W1.9mm_P5.00mm -> Capacitor_THT:C_Disc_D5.0mm_W2.5mm_P2.50mm
- D2: footprint Diode_THT:D_A-405_P7.62mm_Horizontal -> Diode_THT:D_DO-41_SOD81_P7.62mm_Horizontal
- J3: renamed from J1; footprint TerminalBlock:TerminalBlock_bornier-2_P5.08mm -> TerminalBlock_Phoenix:TerminalBlock_Phoenix_MKDS-1,5-2-5.08_1x02_P5.08mm_Horizontal
- R4, R5: footprint Resistor_THT:R_Axial_DIN0207_L6.3mm_D2.5mm_P10.16mm_Horizontal -> Resistor_THT:R_Axial_DIN0207_L6.3mm_D2.5mm_P7.62mm_Horizontal
- TP1, TP2, TP4: footprint (none) -> TestPoint:TestPoint_Loop_D2.50mm_Drill1.0mm
- TP3: renamed from TP5; footprint (none) -> TestPoint:TestPoint_Loop_D2.50mm_Drill1.0mm
- TP5: renamed from TP3; footprint (none) -> TestPoint:TestPoint_Loop_D2.50mm_Drill1.0mm
- renumbered D9 to D8, D8 to D9, J2 to J1, J3 to J2, JP3 to JP2, R13 to R12, R12 to R13
Connections:
- net GND: now also U1.3, U1.5, TP6.1; no longer U1.11, U1.13
- net SCL: no longer TP4.1, U4.14 (RC3/SCK/SCL)
- net at R7.2: now also U1.12; no longer U1.8
- net at R3.1: now also U1.10; no longer U1.6
- net at U1.2, U1.9: now also U1.11, U1.13; no longer U1.3, U1.5
- net at U1.4: no longer R6.2
- net DATA_IN renamed SDO
- new net: R6.2, U1.8
- new net CLK: TP4.1, U4.14 (RC3/SCK/SCL)
- no-connect marks 19 -> 20
Other:
- note removed: "Close to LM358"
- moved on the sheet: D8, H1, H2, H3, H4, H5, H6, H7, Q1, R11, R12, R14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

Commit message: reset
Parts:
- removed TP6: GND, TestPoint:TestPoint_Loop_D2.50mm_Drill1.0mm, symbol Connector:TestPoint
- added C5: 100n, Capacitor_THT:C_Disc_D4.3mm_W1.9mm_P5.00mm, symbol Device:C_Small
- added H10, H11, H12, H8, H9: MountingHole, MountingHole:MountingHole_3.2mm_M3, symbol Mechanical:MountingHole
- added J6: Expr 2, Connector_PinHeader_2.54mm:PinHeader_1x02_P2.54mm_Vertical, symbol Connector:Screw_Terminal_01x02
- added J7: Expr 1, Connector_PinHeader_2.54mm:PinHeader_1x02_P2.54mm_Vertical, symbol Connector:Screw_Terminal_01x02
- added R16, R17: 10, Resistor_THT:R_Axial_DIN0207_L6.3mm_D2.5mm_P10.16mm_Horizontal, symbol Device:R
- added U5: LM358, Package_DIP:CERDIP-8_W7.62mm_SideBrazed_Socket, symbol Amplifier_Operational:LM358
- C1: footprint Capacitor_THT:C_Disc_D5.0mm_W2.5mm_P2.50mm -> Capacitor_THT:C_Disc_D4.3mm_W1.9mm_P5.00mm
- C14: renamed from C3; footprint Capacitor_THT:C_Disc_D5.0mm_W2.5mm_P2.50mm -> Capacitor_THT:C_Disc_D4.3mm_W1.9mm_P5.00mm
- C2: footprint Capacitor_THT:CP_Radial_D6.3mm_P2.50mm -> (none)
- C3: renamed from C4; footprint Capacitor_THT:CP_Radial_D5.0mm_P2.00mm -> (none)
- C4: renamed from C5; footprint Capacitor_THT:C_Disc_D5.0mm_W2.5mm_P2.50mm -> Capacitor_THT:C_Disc_D4.3mm_W1.9mm_P5.00mm
- D2: footprint Diode_THT:D_DO-41_SOD81_P7.62mm_Horizontal -> Diode_THT:D_A-405_P7.62mm_Horizontal
- J1: renamed from J3; footprint TerminalBlock_Phoenix:TerminalBlock_Phoenix_MKDS-1,5-2-5.08_1x02_P5.08mm_Horizontal -> TerminalBlock:TerminalBlock_bornier-2_P5.08mm
- R4, R5: footprint Resistor_THT:R_Axial_DIN0207_L6.3mm_D2.5mm_P7.62mm_Horizontal -> Resistor_THT:R_Axial_DIN0207_L6.3mm_D2.5mm_P10.16mm_Horizontal
- TP1, TP2, TP4: footprint TestPoint:TestPoint_Loop_D2.50mm_Drill1.0mm -> (none)
- TP3: renamed from TP5; footprint TestPoint:TestPoint_Loop_D2.50mm_Drill1.0mm -> (none)
- TP5: renamed from TP3; footprint TestPoint:TestPoint_Loop_D2.50mm_Drill1.0mm -> (none)
- renumbered D9 to D8, D8 to D9, J1 to J2, J2 to J3, JP2 to JP3, R13 to R12, R12 to R13
Connections:
- net CLK is gone; now on net SCL: TP4.1, U4.14 (RC3/SCK/SCL)
- net GND: now also U1.11, U1.13, C5.1, J6.2 (Pin_2), J7.2 (Pin_2), U5.4 (V-); no longer U1.3, U1.5
- net VEE: now also C5.2, U5.8 (V+)
- net at U4.4 (Vref-/AN2/RA2): now also U5.3 (+), U5.5 (+)
- net at R7.2: now also U1.8; no longer U1.12
- net at R3.1: now also U1.6; no longer U1.10
- net at U1.2, U1.9: now also U1.3, U1.5; no longer U1.11, U1.13
- net at U1.4: now also R6.2
- net SDO renamed DATA_IN
- new net: R16.1, U5.6 (-), U5.7
- new net: J6.1 (Pin_1), R16.2
- new net: R17.1, U5.1, U5.2 (-)
- new net: J7.1 (Pin_1), R17.2
- no-connect marks 20 -> 19
Other:
- note added: "Close to LM358"
- moved on the sheet: D9, H1, H2, H3, H4, H5, H6, H7, Q1, R11, R13, R14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
