File: Avrille/64_Outs/64_Outs.kicad_pcb (KiCad board)
At the start: 2 copper layers, 261.6 x 199.4 mm, 341 parts, among them J1 POWER, J2 Midi-In, J3 Midi-Thru, J4 ICSP, J5 FT232, J8 DIN41612_02x32_AC, J9 DIN41612_02x32_AC, Q1 BC337, Q10 SSM3J351R, Q11 SSM3J351R, Q12 SSM3J351R, Q13 SSM3J351R, Q14 SSM3J351R, Q15 SSM3J351R, Q16 SSM3J351R, Q17 SSM3J351R, Q18 SSM3J351R, Q19 SSM3J351R, Q2 SSM3J351R, Q20 SSM3J351R, Q21 SSM3J351R, Q22 SSM3J351R, Q23 SSM3J351R, Q24 SSM3J351R, Q25 SSM3J351R, Q26 SSM3J351R, Q27 SSM3J351R, Q28 SSM3J351R, Q29 SSM3J351R, Q3 SSM3J351R, Q30 SSM3J351R, Q31 SSM3J351R, Q32 SSM3J351R, Q33 SSM3J351R, Q34 SSM3J351R, Q35 SSM3J351R, Q36 SSM3J351R, Q37 SSM3J351R, Q38 SSM3J351R, Q39 SSM3J351R, Q4 SSM3J351R, Q40 SSM3J351R, Q41 SSM3J351R, Q42 SSM3J351R, Q43 SSM3J351R, Q44 SSM3J351R, Q45 SSM3J351R, Q46 SSM3J351R, Q47 SSM3J351R, Q48 SSM3J351R, Q49 SSM3J351R, Q5 SSM3J351R, Q50 SSM3J351R, Q58 SSM3J351R, Q59 SSM3J351R, Q6 SSM3J351R, Q60 SSM3J351R, Q61 SSM3J351R, Q62 SSM3J351R, Q63 SSM3J351R, Q64 SSM3J351R, Q65 SSM3J351R, Q7 SSM3J351R, Q74 SSM3J351R, Q75 SSM3J351R, Q76 SSM3J351R, Q77 SSM3J351R, Q78 SSM3J351R, Q79 SSM3J351R, Q8 SSM3J351R, Q80 SSM3J351R, Q9 SSM3J351R, SW1 RESET, SW2 Prog, SW3 Channel, U1 74HC14, U10 74HC595, U11 74HC595, U12 74HC595, U13 74HC595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

Commit message: Layout for Review
Parts:
- Q10, Q11, Q12, Q13, Q14, Q15, Q16, Q17, Q18, Q19, Q2, Q20, Q21, Q22, Q23, Q24, Q25, Q26, Q27, Q28, Q29, Q3, Q30, Q31, Q32, Q33, Q34, Q35, Q36, Q37, Q38, Q39, Q4, Q40, Q41, Q42, Q43, Q44, Q45, Q46, Q47, Q48, Q49, Q5, Q50, Q58, Q59, Q6, Q60, Q61, Q62, Q63, Q64, Q65, Q7, Q74, Q75, Q76, Q77, Q78, Q79, Q8, Q80, Q9: footprint Package_SO:SOTFL95P240X88-3N -> 64_Outs:SOTFL95P240X88-3N
- moved U15 80.8 mm to (112.7, 175.8)
- moved U19 79.6 mm to (172.7, 175.8)
- moved U20 79.4 mm to (292.7, 175.8)
- moved U16 79.2 mm to (232.7, 175.8)
- moved R29 76.6 mm to (193.0, 192.5), turned to 90 degrees
- moved R21 76.0 mm to (193.0, 189.3), turned to -90 degrees
- moved R117 75.6 mm to (187.7, 192.5), turned to 90 degrees
- moved R26 75.3 mm to (252.9, 192.5), turned to 90 degrees
- moved R18 74.7 mm to (252.9, 189.3), turned to -90 degrees
- moved R114 74.5 mm to (247.7, 192.5), turned to 90 degrees
- moved R25 74.5 mm to (133.0, 192.5), turned to 90 degrees
- moved R113 73.9 mm to (127.7, 192.5), turned to 90 degrees
- moved R17 73.9 mm to (133.0, 189.3), turned to -90 degrees
- moved R118 73.8 mm to (307.7, 192.5), turned to 90 degrees
- moved R30 73.5 mm to (312.9, 192.5), turned to 90 degrees
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Connections:
- R56 pad 1: unconnected-(R56-Pad1) -> /Module_33/Sorties_8/Cmd_3
- R57 pad 1: unconnected-(R57-Pad1) -> /Module_32/Sorties_9/Cmd_3
- R58 pad 1: unconnected-(R58-Pad1) -> /Module_33/Sorties_9/Cmd_3
- R59 pad 1: unconnected-(R59-Pad1) -> /Module_32/Sorties_10/Cmd_3
- R60 pad 1: unconnected-(R60-Pad1) -> /Module_33/Sorties_10/Cmd_3
- R61 pad 1: unconnected-(R61-Pad1) -> /Module_32/Sorties_11/Cmd_3
- R62 pad 1: unconnected-(R62-Pad1) -> /Module_33/Sorties_11/Cmd_3
- R63 pad 1: unconnected-(R63-Pad1) -> /Module_32/Sorties_8/Cmd_3
Routing:
- net /Module_32/Sorties_10/V_IN: track 67.8 -> 456.1 mm, vias 0 -> 32
- net /Module_33/Sorties_10/V_IN: track 67.8 -> 452.4 mm, vias 0 -> 32
- net /~{OE}: track 0.00 -> 291.8 mm, vias 0 -> 9
- net /LAT: track 0.00 -> 277.9 mm, vias 0 -> 8
- net /SCL: track 0.00 -> 271.5 mm, vias 0 -> 8
- net GND: track 76.2 -> 339.2 mm, vias 0 -> 347
- net VCC: track 477.9 -> 673.3 mm
- net /DATA_IN: track 0.00 -> 152.5 mm, vias 0 -> 1
- net /Module_33/O_07: track 0.00 -> 77.2 mm, vias 0 -> 1
- net /TxD: track 0.00 -> 75.1 mm, vias 0 -> 1
- net /Module_33/O_06: track 0.00 -> 74.4 mm, vias 0 -> 1
- net /RxD: track 0.00 -> 73.0 mm, vias 0 -> 1
- net /Module_33/O_00: track 0.00 -> 72.7 mm, vias 0 -> 1
- net /Module_33/O_05: track 0.00 -> 71.4 mm, vias 0 -> 1
- net /Module_33/O_01: track 0.00 -> 69.5 mm, vias 0 -> 1
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- added copper zone on B.Cu, net GND
- added copper zone on F.Cu, net GND
