File: Avrille/64_Outs/Sorties_8.kicad_sch (KiCad schematic)
At the start: 33 parts, among them Q2 SSM3J351R, Q3 SSM3J351R, Q5 SSM3J351R, Q6 SSM3J351R, Q7 SSM3J351R, Q74 SSM3J351R, Q8 SSM3J351R, Q9 SSM3J351R, U14 ULN2803A

Commit message: Layout for Review
Parts:
- Q2, Q3, Q5, Q6, Q7, Q74, Q8, Q9: footprint SOTFL95P240X88-3N -> 64_Outs:SOTFL95P240X88-3N
Connections:
- net Cmd_3: now also R56.1
Changed lines of the file:
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@@
 	(wire
 		(pts
-			(xy 152.4 111.76) (xy 154.94 111.76)
+			(xy 151.13 111.76) (xy 154.94 111.76)
 		)
 		(stroke
@@
 	(wire
 		(pts
-			(xy 86.36 60.96) (xy 88.9 60.96)
+			(xy 86.36 60.96) (xy 90.17 60.96)
 		)
 		(stroke
@@
 	)
 	(label "Cmd_6"
-		(at 152.4 111.76 180)
+		(at 151.13 111.76 180)
 		(effects
 			(font
@@
 			)
 		)
-		(property "Footprint" "SOTFL95P240X88-3N"
+		(property "Footprint" "64_Outs:SOTFL95P240X88-3N"
 			(at 240.03 159.69 0)
 			(effects
@@
 			)
 		)
-		(property "Footprint" "SOTFL95P240X88-3N"
+		(property "Footprint" "64_Outs:SOTFL95P240X88-3N"
 			(at 242.57 210.49 0)
 			(effects
@@
 			)
 		)
-		(property "Footprint" "SOTFL95P240X88-3N"
+		(property "Footprint" "64_Outs:SOTFL95P240X88-3N"
 			(at 179.07 210.49 0)
 			(effects
@@
 			)
 		)
-		(property "Footprint" "SOTFL95P240X88-3N"
+		(property "Footprint" "64_Outs:SOTFL95P240X88-3N"
 			(at 176.53 159.69 0)
 			(effects
@@
 			)
 		)
-		(property "Footprint" "SOTFL95P240X88-3N"
+		(property "Footprint" "64_Outs:SOTFL95P240X88-3N"
 			(at 52.07 210.49 0)
 			(effects
@@
 			)
 		)
-		(property "Footprint" "SOTFL95P240X88-3N"
+		(property "Footprint" "64_Outs:SOTFL95P240X88-3N"
 			(at 113.03 159.69 0)
 			(effects
@@
 			)
 		)
-		(property "Footprint" "SOTFL95P240X88-3N"
+		(property "Footprint" "64_Outs:SOTFL95P240X88-3N"
 			(at 49.53 159.69 0)
 			(effects
@@
 			)
 		)
-		(property "Footprint" "SOTFL95P240X88-3N"
+		(property "Footprint" "64_Outs:SOTFL95P240X88-3N"
 			(at 115.57 210.49 0)
 			(effects
